File: hardware/ML8511_Breakout.brd (EAGLE design)
At the start: 15.2 x 15.2 mm, 11 parts, among them U1 ML8511-UV-SENSOR

Commit message: added local fiducials
Parts:
- added FID1, FID2: FIDUCIAL1X2, SparkFun-Aesthetics:FIDUCIAL-1X2
